Commit message: new commit

File: mobilearmbot_description/urdf/mobile_base.xacro (robot description, xacro)
@@ -21,5 +21,4 @@
                 </geometry>
                 <origin xyz="0 0 0" rpy="${pi / 2.0} 0 0"/>
-                <material name="grey"/>
             </collision>
             <xacro:cylinder_inertia m="1.0" r="${2*wheel_radius}" h="${2*wheel_length}"
@@ -60,5 +59,4 @@
             </geometry>
             <origin xyz="0 0 0" rpy="0 0 0"/>
-            <material name="grey"/>
         </collision>
         <xacro:sphere_inertia m="0.5" r="${2*caster_wheel_radius}"
