Commit message: update

File: mobilearmbot_description/urdf/arm.xacro (robot description, xacro)
@@ -27,6 +27,6 @@
                 <origin xyz="0 0 ${arm_length/2.0}" rpy="0 0 0"/>
             </collision>
-            <xacro:cylinder_inertia m="0.3" r="${arm_radius}" h="${arm_length}"
-                                    xyz="0 0 0" rpy="0 0 0"/>
+            <xacro:cylinder_inertia m="0.3" r="${2*arm_radius}" h="${2*arm_length}"
+                                    xyz="0 0 ${arm_length/2.0}" rpy="0 0 0"/>
         </link>
     </xacro:macro>
@@ -46,6 +46,6 @@
             </geometry>
         </collision>
-        <xacro:cylinder_inertia m="0.5" r="${arm_base_radius}" h="${arm_base_length}"
-                                xyz="0 0 0" rpy="0 0 0"/>
+        <xacro:cylinder_inertia m="0.5" r="${2*arm_base_radius}" h="${2*arm_base_length}"
+                                xyz="0 0 ${arm_base_length/2.0}" rpy="0 0 0"/>
     </link>
     <xacro:arm_link link_name="forearm" color="yellow"/>

File: mobilearmbot_description/urdf/mobilearmbot.urdf.xacro (robot description, xacro)
@@ -10,5 +10,5 @@
         <parent link="base_link"/>
         <child link="arm_base_link"/>
-        <origin xyz="${base_length/3.0} 0 ${base_height}" rpy="0 0 0"/>
+        <origin xyz="${base_length/4.0} 0 ${base_height}" rpy="0 0 0"/>
     </joint>
 </robot>
